Commit message: Base of the manipulator

File: src/mani_gz_sim/description/robot.urdf.xacro (robot description, xacro)
@@ -2,5 +2,5 @@
 <robot xmlns:xacro="http://www.ros.org/wiki/xacro"  name="robot">
     <xacro:include filename="robot_core.xacro" />
-    <xacro:include filename="gazebo_control.xacro" />
-    <xacro:include filename="lidar.xacro" />
+    <!-- <xacro:include filename="gazebo_control.xacro" /> -->
+    <!-- <xacro:include filename="lidar.xacro" /> -->
 </robot>

File: src/mani_gz_sim/description/robot_core.xacro (robot description, xacro)
@@ -2,30 +2,32 @@
 <robot xmlns:xacro="http://www.ros.org/wiki/xacro" >
     <xacro:include filename="inertial_macros.xacro"/>
-    <material name="white">
-        <color rgba="1 1 1 1" />
-    </material>
-    <material name="purple">
-        <color rgba="0.0 0.0 0.1 1"/>
-    </material>
-     <material name="grey">
-        <color rgba="0.2 0.2 0.2 1"/>
-    </material>
-     <material name="dark_blue">
-        <color rgba="0.0 0.0 0.5 1"/>
-    </material>
-    <material name="blue">
-        <color rgba="0.2 0.1 0.2 1"/>
-    </material>
-   <material name="red">
-        <color rgba="0.2 0.0 0.0 1"/>
-    </material>
-    <material name="black2">
-        <color rgba="0 0 0 1"/>
-    </material>
+    <xacro:include filename="colors.xacro"/>
     <!-- BASE LINK -->
     <link name="base_link">
+        <visual>
+            <origin xyz="0 0 0"/>
+            <geometry>
+                <cylinder radius="0.3" length="0.1"/>
+            </geometry>
+            <material name="black"/>
+        </visual>
+        <visual>
+            <origin xyz="0 0 0"/>
+            <geometry>
+                <cylinder radius="0.3" length="0.1"/>
+            </geometry>
+            <material name="black"/>
+        </visual>
+        <collision>
+            <origin xyz="0 0 0"/>
+            <geometry>
+                <cylinder radius="0.3" length="0.1"/>
+            </geometry>
+        </collision>
+        <xacro:inertial_cylinder mass="0.5" radius="0.3" length="0.1">
+            <origin xyz="0 0 0" rpy="0 0 0"/>
+        </xacro:inertial_cylinder>
     </link>
-    <!-- CHASSIS LINK -->
-     <joint name="chassis_joint" type="fixed">
+    <joint name="base_link_2" type="fixed">
         <parent link="base_link"/>
         <child link="chassis"/>
@@ -34,137 +36,24 @@
     <link name="chassis">
         <visual>
-            <origin xyz="0 0 0.11"/> <!-- połowa dlugosci chessis plis polowa kola 0.075 + 0.035-->
+            <origin xyz="0 0 0.1"/>
             <geometry>
-                <box size="0.3 0.2 0.15"/>
+                <cylinder radius="0.25" length="0.5"/>
+            </geometry>
+            <material name="blue"/>
+        </visual>
+        <visual>
+            <origin xyz="0 0 0.1"/>
+            <geometry>
+                <cylinder radius="0.25" length="0.5"/>
             </geometry>
             <material name="blue"/>
         </visual>
         <collision>
-            <origin xyz="0 0 0.11"/>
+            <origin xyz="0 0 0.1"/>
             <geometry>
-                <box size="0.3 0.2 0.15"/>
+                <cylinder radius="0.25" length="0.5"/>
             </geometry>
         </collision>
-        <xacro:inertial_box mass="0.5" x="0.3" y="0.2" z="0.15">
-            <origin xyz="0 0 0.11" rpy="0 0 0"/>
-        </xacro:inertial_box>
-    </link>
-    <joint name="puck_joint" type="fixed">
-        <parent link="chassis"/>
-        <child link="puck"/>
-        <origin xyz="0 0 0.19"/>
-    </joint>
-    <link name="puck">
-        <visual>
-            <geometry>
-                <cylinder radius="0.03" length="0.01"/>
-            </geometry>
-            <material name="black"/>
-        </visual>
-         <visual>
-            <origin xyz="0 0 -0.05"/>
-            <geometry>
-                <cylinder radius="0.03" length="0.01"/>
-            </geometry>
-            <material name="black"/>
-        </visual>
-        <collision>
-            <geometry>
-                <cylinder radius="0.03" length="0.01"/>
-            </geometry>
-        </collision>
-        <xacro:inertial_cylinder mass="0.1" length="0.01" radius="0.03">
-            <origin xyz="0 0 0" rpy="0 0 0"/>
-        </xacro:inertial_cylinder>
-    </link>
-    <!-- LEFT DOWN WHEEL LINK -->
-    <joint name="left_down_wheel_joint" type="continuous">
-        <parent link="base_link"/>
-        <child link="left_down_wheel"/>
-        <origin xyz="-0.08 0.115 0.035" rpy="-${pi/2} 0 0" />
-        <axis xyz="0 0 1"/>
-    </joint>
-    <link name="left_down_wheel">
-        <visual>
-            <geometry>
-                <cylinder radius="0.035" length="0.03"/>
-            </geometry>
-            <material name="black2"/>
-        </visual>
-        <collision>
-            <geometry>
-                <cylinder radius="0.035" length="0.03"/>
-            </geometry>
-        </collision>
-        <xacro:inertial_cylinder mass="0.1" length="0.03" radius="0.035">
-            <origin xyz="0 0 0" rpy="0 0 0"/>
-        </xacro:inertial_cylinder>
-    </link>
-    <!-- RIGHT DOWN WHEEL LINK -->
-    <joint name="right_down_wheel_joint" type="continuous">
-        <parent link="base_link"/>
-        <child link="right_down_wheel"/>
-        <origin xyz="0.08 -0.115 0.035" rpy="${pi/2} 0 0" />
-        <axis xyz="0 0 -1"/>
-    </joint>
-    <link name="right_down_wheel">
-        <visual>
-            <geometry>
-                <cylinder radius="0.035" length="0.03"/>
-            </geometry>
-            <material name="black2"/>
-        </visual>
-        <collision>
-            <geometry>
-                <cylinder radius="0.035" length="0.03"/>
-            </geometry>
-        </collision>
-        <xacro:inertial_cylinder mass="0.1" length="0.03" radius="0.035">
-            <origin xyz="0 0 0" rpy="0 0 0"/>
-        </xacro:inertial_cylinder>
-    </link>
-    <!-- LEFT UP WHEEL LINK -->
-    <joint name="left_up_wheel_joint" type="continuous">
-        <parent link="base_link"/>
-        <child link="left_up_wheel"/>
-        <origin xyz="0.08 0.115 0.035" rpy="-${pi/2} 0 0" />
-        <axis xyz="0 0 1"/>
-    </joint>
-    <link name="left_up_wheel">
-        <visual>
-            <geometry>
-                <cylinder radius="0.035" length="0.03"/>
-            </geometry>
-            <material name="black2"/>
-        </visual>
-        <collision>
-            <geometry>
-                <cylinder radius="0.035" length="0.03"/>
-            </geometry>
-        </collision>
-        <xacro:inertial_cylinder mass="0.1" length="0.03" radius="0.035">
-            <origin xyz="0 0 0" rpy="0 0 0"/>
-        </xacro:inertial_cylinder>
-    </link>
-    <!-- RIGHT UP WHEEL LINK -->
-    <joint name="right_up_wheel_joint" type="continuous">
-        <parent link="base_link"/>
-        <child link="right_up_wheel"/>
-        <origin xyz="-0.08 -0.115 0.035" rpy="${pi/2} 0 0" />
-        <axis xyz="0 0 -1"/>
-    </joint>
-    <link name="right_up_wheel">
-        <visual>
-            <geometry>
-                <cylinder radius="0.035" length="0.03"/>
-            </geometry>
-            <material name="black2"/>
-        </visual>
-        <collision>
-            <geometry>
-                <cylinder radius="0.035" length="0.03"/>
-            </geometry>
-        </collision>
-        <xacro:inertial_cylinder mass="0.1" length="0.03" radius="0.035">
+        <xacro:inertial_cylinder mass="0.5" radius="0.25" length="0.5">
             <origin xyz="0 0 0" rpy="0 0 0"/>
         </xacro:inertial_cylinder>
