Commit message: Another try to move the two joint ended failure

File: src/mani_gz_sim/description/colors.xacro (robot description, xacro)
@@ -22,3 +22,6 @@
         <color rgba="0 0 0 1"/>
     </material>
+    <material name="black">
+    <color rgba="0 0 0 1"/>
+</material>
 </robot>

File: src/mani_gz_sim/description/gazebo_control.xacro (robot description, xacro)
@@ -26,8 +26,9 @@
     </ros2_control>
     <!-- Gazebo Sim plugin -->
+    <!-- Gazebo Sim plugin -->
     <gazebo>
         <plugin
-            name="gz_ros2_control::GazeboSimROS2ControlPlugin"
-            filename="libgz_ros2_control-system">
+            filename="libgz_ros2_control-system.so"
+            name="gz_ros2_control::GazeboSimROS2ControlPlugin">
             <parameters>
                 $(find mani_gz_sim)/config/controllers.yaml

File: src/mani_gz_sim/description/robot_core.xacro (robot description, xacro)
@@ -22,8 +22,11 @@
         </xacro:inertial_cylinder>
     </link>
-    <joint name="joint_1" type="fixed">
+    <joint name="joint_1" type="revolute">
         <parent link="base_link"/>
         <child link="platform"/>
         <origin xyz="0 0 0"/>
+        <axis xyz="0 0 1"/>
+        <limit lower="-3.14159" upper="3.14159"
+           effort="10" velocity="1.0"/>
     </joint>
     <link name="platform">
@@ -45,8 +48,11 @@
         </xacro:inertial_cylinder>
     </link>
-    <joint name="joint_2" type="fixed">
+    <joint name="joint_2" type="revolute">
         <parent link="platform"/>
         <child link="circuit_joint"/>
         <origin xyz="0 0 0"/>
+        <axis xyz="0 0 1"/>
+        <limit lower="-3.14159" upper="3.14159"
+           effort="10" velocity="1.0"/>
     </joint>
     <link name="circuit_joint">
