Commit message: The designed base of the modulator, without motion

File: src/mani_gz_sim/description/robot_core.xacro (robot description, xacro)
@@ -8,12 +8,5 @@
             <origin xyz="0 0 0"/>
             <geometry>
-                <cylinder radius="0.3" length="0.1"/>
-            </geometry>
-            <material name="black"/>
-        </visual>
-        <visual>
-            <origin xyz="0 0 0"/>
-            <geometry>
-                <cylinder radius="0.3" length="0.1"/>
+                <cylinder radius="0.5" length="0.1"/>
             </geometry>
             <material name="black"/>
@@ -22,39 +15,78 @@
             <origin xyz="0 0 0"/>
             <geometry>
-                <cylinder radius="0.3" length="0.1"/>
+                <cylinder radius="0.5" length="0.1"/>
             </geometry>
         </collision>
-        <xacro:inertial_cylinder mass="0.5" radius="0.3" length="0.1">
+        <xacro:inertial_cylinder mass="0.5" radius="0.5" length="0.1">
             <origin xyz="0 0 0" rpy="0 0 0"/>
         </xacro:inertial_cylinder>
     </link>
-    <joint name="base_link_2" type="fixed">
+    <joint name="joint_1" type="fixed">
         <parent link="base_link"/>
-        <child link="chassis"/>
+        <child link="platform"/>
         <origin xyz="0 0 0"/>
     </joint>
-    <link name="chassis">
+    <link name="platform">
         <visual>
-            <origin xyz="0 0 0.1"/>
+            <origin xyz="0 0 0.2"/>
             <geometry>
-                <cylinder radius="0.25" length="0.5"/>
-            </geometry>
-            <material name="blue"/>
-        </visual>
-        <visual>
-            <origin xyz="0 0 0.1"/>
-            <geometry>
-                <cylinder radius="0.25" length="0.5"/>
+                <cylinder radius="0.45" length="0.3"/>
             </geometry>
             <material name="blue"/>
         </visual>
         <collision>
-            <origin xyz="0 0 0.1"/>
+            <origin xyz="0 0 0.2"/>
             <geometry>
-                <cylinder radius="0.25" length="0.5"/>
+                <cylinder radius="0.45" length="0.3"/>
             </geometry>
         </collision>
-        <xacro:inertial_cylinder mass="0.5" radius="0.25" length="0.5">
-            <origin xyz="0 0 0" rpy="0 0 0"/>
+        <xacro:inertial_cylinder mass="0.5" radius="0.45" length="0.3">
+            <origin xyz="0 0 0.2" rpy="0 0 0"/>
+        </xacro:inertial_cylinder>
+    </link>
+    <joint name="joint_2" type="fixed">
+        <parent link="platform"/>
+        <child link="circuit_joint"/>
+        <origin xyz="0 0 0"/>
+    </joint>
+    <link name="circuit_joint">
+        <visual>
+            <origin xyz="0 0 0.35" rpy="0 1.5708 0"/>
+            <geometry>
+                <cylinder radius="0.3" length="0.45"/>
+            </geometry>
+            <material name="purple"/>
+        </visual>
+        <collision>
+            <origin xyz="0 0 0.35" rpy="0 1.5708 0"/>
+            <geometry>
+                <cylinder radius="0.3" length="0.45"/>
+            </geometry>
+        </collision>
+        <xacro:inertial_cylinder mass="0.5" radius="0.3" length="0.45">
+            <origin xyz="0 0 0.35" rpy="0 1.5708 0"/>
+        </xacro:inertial_cylinder>
+    </link>
+    <joint name="joint_3" type="fixed">
+        <parent link="circuit_joint"/>
+        <child link="arm_1"/>
+        <origin xyz="0 0 0"/>
+    </joint>
+    <link name="arm_1">
+        <visual>
+            <origin xyz="0 0 1.1"/>
+            <geometry>
+                <cylinder radius="0.2" length="1.1"/>
+            </geometry>
+            <material name="white"/>
+        </visual>
+        <collision>
+            <origin xyz="0 0 1.1"/>
+            <geometry>
+                <cylinder radius="0.2" length="1.1"/>
+            </geometry>
+        </collision>
+        <xacro:inertial_cylinder mass="0.5" radius="0.2" length="1.1">
+            <origin xyz="0 0 1.1"/>
         </xacro:inertial_cylinder>
     </link>

Commit message: Added basic movement of the first joints

File: src/mani_gz_sim/description/robot_core.xacro (robot description, xacro)
@@ -18,5 +18,5 @@
             </geometry>
         </collision>
-        <xacro:inertial_cylinder mass="0.5" radius="0.5" length="0.1">
+        <xacro:inertial_cylinder mass="2.0" radius="0.5" length="0.1">
             <origin xyz="0 0 0" rpy="0 0 0"/>
         </xacro:inertial_cylinder>
@@ -44,15 +44,12 @@
             </geometry>
         </collision>
-        <xacro:inertial_cylinder mass="0.5" radius="0.45" length="0.3">
+        <xacro:inertial_cylinder mass="1" radius="0.45" length="0.3">
             <origin xyz="0 0 0.2" rpy="0 0 0"/>
         </xacro:inertial_cylinder>
     </link>
-    <joint name="joint_2" type="revolute">
+    <joint name="joint_2_fixed" type="fixed">
         <parent link="platform"/>
         <child link="circuit_joint"/>
         <origin xyz="0 0 0"/>
-        <axis xyz="0 0 1"/>
-        <limit lower="-3.14159" upper="3.14159"
-           effort="10" velocity="1.0"/>
     </joint>
     <link name="circuit_joint">
@@ -74,12 +71,15 @@
         </xacro:inertial_cylinder>
     </link>
-    <joint name="joint_3" type="fixed">
+    <joint name="joint_2" type="revolute">
         <parent link="circuit_joint"/>
         <child link="arm_1"/>
         <origin xyz="0 0 0"/>
+        <axis xyz="1 0 0"/>
+        <limit lower="-3.14159" upper="3.14159"
+           effort="10" velocity="1.0"/>
     </joint>
     <link name="arm_1">
         <visual>
-            <origin xyz="0 0 1.1"/>
+            <origin xyz="0 0 1.2"/>
             <geometry>
                 <cylinder radius="0.2" length="1.1"/>
@@ -88,10 +88,10 @@
         </visual>
         <collision>
-            <origin xyz="0 0 1.1"/>
+            <origin xyz="0 0 1.2"/>
             <geometry>
                 <cylinder radius="0.2" length="1.1"/>
             </geometry>
         </collision>
-        <xacro:inertial_cylinder mass="0.5" radius="0.2" length="1.1">
+        <xacro:inertial_cylinder mass="0.5" radius="0.2" length="1.2">
             <origin xyz="0 0 1.1"/>
         </xacro:inertial_cylinder>

Commit message: Working joint_2

File: src/mani_gz_sim/description/robot_core.xacro (robot description, xacro)
@@ -18,5 +18,5 @@
             </geometry>
         </collision>
-        <xacro:inertial_cylinder mass="2.0" radius="0.5" length="0.1">
+        <xacro:inertial_cylinder mass="10.0" radius="0.5" length="0.1">
             <origin xyz="0 0 0" rpy="0 0 0"/>
         </xacro:inertial_cylinder>
@@ -44,16 +44,19 @@
             </geometry>
         </collision>
-        <xacro:inertial_cylinder mass="1" radius="0.45" length="0.3">
+        <xacro:inertial_cylinder mass="3.0" radius="0.45" length="0.3">
             <origin xyz="0 0 0.2" rpy="0 0 0"/>
         </xacro:inertial_cylinder>
     </link>
-    <joint name="joint_2_fixed" type="fixed">
+    <joint name="joint_2" type="revolute">
         <parent link="platform"/>
         <child link="circuit_joint"/>
-        <origin xyz="0 0 0"/>
+        <origin xyz="0 0 0.35" rpy="0 0 0"/>
+        <axis xyz="1 0 0"/>
+        <limit lower="-3.14159" upper="3.14159"
+           effort="10" velocity="1.0"/>
     </joint>
     <link name="circuit_joint">
         <visual>
-            <origin xyz="0 0 0.35" rpy="0 1.5708 0"/>
+            <origin xyz="0 0 0" rpy="0 1.5708 0"/>
             <geometry>
                 <cylinder radius="0.3" length="0.45"/>
@@ -62,37 +65,34 @@
         </visual>
         <collision>
-            <origin xyz="0 0 0.35" rpy="0 1.5708 0"/>
+            <origin xyz="0 0 0" rpy="0 1.5708 0"/>
             <geometry>
                 <cylinder radius="0.3" length="0.45"/>
             </geometry>
         </collision>
-        <xacro:inertial_cylinder mass="0.5" radius="0.3" length="0.45">
-            <origin xyz="0 0 0.35" rpy="0 1.5708 0"/>
+        <xacro:inertial_cylinder mass="2.0" radius="0.3" length="0.45">
+            <origin xyz="0 0 0" rpy="0 1.5708 0"/>
         </xacro:inertial_cylinder>
     </link>
-    <joint name="joint_2" type="revolute">
+    <joint name="joint_2_fixed" type="fixed">
         <parent link="circuit_joint"/>
         <child link="arm_1"/>
         <origin xyz="0 0 0"/>
-        <axis xyz="1 0 0"/>
-        <limit lower="-3.14159" upper="3.14159"
-           effort="10" velocity="1.0"/>
     </joint>
     <link name="arm_1">
         <visual>
-            <origin xyz="0 0 1.2"/>
+            <origin xyz="0 0 0.8" rpy="0 0 0"/>
             <geometry>
-                <cylinder radius="0.2" length="1.1"/>
+                <cylinder radius="0.1" length="1.1"/>
             </geometry>
             <material name="white"/>
         </visual>
         <collision>
-            <origin xyz="0 0 1.2"/>
+            <origin xyz="0 0 0.8" rpy="0 0 0"/>
             <geometry>
-                <cylinder radius="0.2" length="1.1"/>
+                <cylinder radius="0.1" length="1.1"/>
             </geometry>
         </collision>
-        <xacro:inertial_cylinder mass="0.5" radius="0.2" length="1.2">
-            <origin xyz="0 0 1.1"/>
+        <xacro:inertial_cylinder mass="0.2" radius="0.1" length="1.2">
+            <origin xyz="0 0 0.8" rpy="0 0 0"/>
         </xacro:inertial_cylinder>
     </link>
