Commit message: First version of robot finished
What was made:
- all three arms and their joints
- basic movement

Want to de:
- improve the build
- add sensor
- made the environment

File: src/mani_gz_sim/description/gazebo_control.xacro (robot description, xacro)
@@ -6,6 +6,5 @@
             <plugin>gz_ros2_control/GazeboSimSystem</plugin>
         </hardware>
-        <!-- First rotating joint -->
-        <joint name="joint_1">
+        <joint name="platform_joint">
             <command_interface name="position">
                 <param name="min">-3.14159</param>
@@ -15,9 +14,24 @@
             <state_interface name="velocity"/>
         </joint>
-        <!-- Second rotating joint -->
-        <joint name="joint_2">
+        <joint name="arm_joint_1">
             <command_interface name="position">
-                <param name="min">-3.14159</param>
-                <param name="max">3.14159</param>
+                <param name="min">-1.047</param>
+                <param name="max">1.047</param>
+            </command_interface>
+            <state_interface name="position"/>
+            <state_interface name="velocity"/>
+        </joint>
+        <joint name="arm_joint_2">
+            <command_interface name="position">
+                <param name="min">-1.5708</param>
+                <param name="max">1.5708</param>
+            </command_interface>
+            <state_interface name="position"/>
+            <state_interface name="velocity"/>
+        </joint>
+        <joint name="arm_joint_3">
+            <command_interface name="position">
+                <param name="min">-1.5708</param>
+                <param name="max">1.5708</param>
             </command_interface>
             <state_interface name="position"/>

File: src/mani_gz_sim/description/robot_core.xacro (robot description, xacro)
@@ -3,5 +3,5 @@
     <xacro:include filename="inertial_macros.xacro"/>
     <xacro:include filename="colors.xacro"/>
-    <!-- BASE LINK -->
+    <!-- =========== BASE LINK =========== -->
     <link name="base_link">
         <visual>
@@ -22,8 +22,8 @@
         </xacro:inertial_cylinder>
     </link>
-    <joint name="joint_1" type="revolute">
+    <joint name="platform_joint" type="revolute">
         <parent link="base_link"/>
         <child link="platform"/>
-        <origin xyz="0 0 0"/>
+        <origin xyz="0 0 0.2"/>
         <axis xyz="0 0 1"/>
         <limit lower="-3.14159" upper="3.14159"
@@ -32,12 +32,12 @@
     <link name="platform">
         <visual>
-            <origin xyz="0 0 0.2"/>
+            <origin xyz="0 0 0"/>
             <geometry>
                 <cylinder radius="0.45" length="0.3"/>
             </geometry>
-            <material name="blue"/>
-        </visual>
-        <collision>
-            <origin xyz="0 0 0.2"/>
+            <material name="black"/>
+        </visual>
+        <collision>
+            <origin xyz="0 0 0"/>
             <geometry>
                 <cylinder radius="0.45" length="0.3"/>
@@ -45,54 +45,155 @@
         </collision>
         <xacro:inertial_cylinder mass="3.0" radius="0.45" length="0.3">
-            <origin xyz="0 0 0.2" rpy="0 0 0"/>
-        </xacro:inertial_cylinder>
-    </link>
-    <joint name="joint_2" type="revolute">
+            <origin xyz="0 0 0" rpy="0 0 0"/>
+        </xacro:inertial_cylinder>
+    </link>
+    <!-- =========== BOTTOM ARM =========== -->
+    <joint name="arm_joint_1" type="revolute">
         <parent link="platform"/>
-        <child link="circuit_joint"/>
-        <origin xyz="0 0 0.35" rpy="0 0 0"/>
+        <child link="circuit_joint_1"/>
+        <origin xyz="0 0 0.15" rpy="0 0 0"/> <!-- platform/2 0.3/2 -->
         <axis xyz="1 0 0"/>
-        <limit lower="-3.14159" upper="3.14159"
+        <limit lower="-1.047" upper="1.047"
+           effort="10" velocity="1.0"/> <!-- pi/3 -->
+    </joint>
+    <link name="circuit_joint_1">
+        <visual>
+            <origin xyz="0 0 0" rpy="0 1.5708 0"/>
+            <geometry>
+                <cylinder radius="0.3" length="0.45"/>
+            </geometry>
+            <material name="white"/>
+        </visual>
+        <collision>
+            <origin xyz="0 0 0" rpy="0 1.5708 0"/>
+            <geometry>
+                <cylinder radius="0.3" length="0.45"/>
+            </geometry>
+        </collision>
+        <xacro:inertial_cylinder mass="2.0" radius="0.3" length="0.45">
+            <origin xyz="0 0 0" rpy="0 1.5708 0"/>
+        </xacro:inertial_cylinder>
+    </link>
+    <joint name="arm_joint_1_fixed" type="fixed">
+        <parent link="circuit_joint_1"/>
+        <child link="arm_1"/>
+        <origin xyz="0 0 0.65"/> <!-- circuit_joint_1/2 0.3/2 + arm_1/2 1.1/2 -->
+    </joint>
+    <link name="arm_1">
+        <visual>
+            <origin xyz="0 0 0" rpy="0 0 0"/>
+            <geometry>
+                <cylinder radius="0.1" length="1.1"/>
+            </geometry>
+            <material name="white"/>
+        </visual>
+        <collision>
+            <origin xyz="0 0 0" rpy="0 0 0"/>
+            <geometry>
+                <cylinder radius="0.1" length="1.1"/>
+            </geometry>
+        </collision>
+        <xacro:inertial_cylinder mass="0.1" radius="0.1" length="1.1">
+            <origin xyz="0 0 0" rpy="0 0 0"/>
+        </xacro:inertial_cylinder>
+    </link>
+    <!-- =========== MIDDLE ARM =========== -->
+    <joint name="arm_joint_2" type="revolute">
+        <parent link="arm_1"/>
+        <child link="circuit_joint_2"/>
+        <origin xyz="0 0 0.55" rpy="0 0 0"/>  <!-- arm_1/2 1.1/2-->
+        <axis xyz="1 0 0"/>
+        <limit lower="-2.356" upper="2.356"
            effort="10" velocity="1.0"/>
     </joint>
-    <link name="circuit_joint">
-        <visual>
-            <origin xyz="0 0 0" rpy="0 1.5708 0"/>
-            <geometry>
-                <cylinder radius="0.3" length="0.45"/>
-            </geometry>
-            <material name="purple"/>
-        </visual>
-        <collision>
-            <origin xyz="0 0 0" rpy="0 1.5708 0"/>
-            <geometry>
-                <cylinder radius="0.3" length="0.45"/>
-            </geometry>
-        </collision>
-        <xacro:inertial_cylinder mass="2.0" radius="0.3" length="0.45">
-            <origin xyz="0 0 0" rpy="0 1.5708 0"/>
-        </xacro:inertial_cylinder>
-    </link>
-    <joint name="joint_2_fixed" type="fixed">
-        <parent link="circuit_joint"/>
-        <child link="arm_1"/>
-        <origin xyz="0 0 0"/>
-    </joint>
-    <link name="arm_1">
-        <visual>
-            <origin xyz="0 0 0.8" rpy="0 0 0"/>
-            <geometry>
-                <cylinder radius="0.1" length="1.1"/>
-            </geometry>
-            <material name="white"/>
-        </visual>
-        <collision>
-            <origin xyz="0 0 0.8" rpy="0 0 0"/>
-            <geometry>
-                <cylinder radius="0.1" length="1.1"/>
-            </geometry>
-        </collision>
-        <xacro:inertial_cylinder mass="0.2" radius="0.1" length="1.2">
-            <origin xyz="0 0 0.8" rpy="0 0 0"/>
+    <link name="circuit_joint_2">
+        <visual>
+            <origin xyz="0 0 0" rpy="0 1.5708 0"/>
+            <geometry>
+                <cylinder radius="0.2" length="0.3"/>
+            </geometry>
+            <material name="blue"/>
+        </visual>
+        <collision>
+            <origin xyz="0 0 0" rpy="0 1.5708 0"/>
+            <geometry>
+                <cylinder radius="0.2" length="0.3"/>
+            </geometry>
+        </collision>
+        <xacro:inertial_cylinder mass="0.1" radius="0.2" length="0.3">
+            <origin xyz="0 0 0" rpy="0 1.5708 0"/>
+        </xacro:inertial_cylinder>
+    </link>
+    <joint name="arm_joint_2_fixed" type="fixed">
+        <parent link="circuit_joint_2"/>
+        <child link="arm_2"/>
+        <origin xyz="0 0 0.65"/> <!-- circuit_joint_2/2 0.2/2 + arm_2/2 1.1/2-->
+    </joint>
+    <link name="arm_2">
+        <visual>
+            <origin xyz="0 0 0" rpy="0 0 0"/>
+            <geometry>
+                <cylinder radius="0.1" length="1.1"/>
+            </geometry>
+            <material name="blue"/>
+        </visual>
+        <collision>
+            <origin xyz="0 0 0" rpy="0 0 0"/>
+            <geometry>
+                <cylinder radius="0.1" length="1.1"/>
+            </geometry>
+        </collision>
+        <xacro:inertial_cylinder mass="0.1" radius="0.1" length="1.2">
+            <origin xyz="0 0 0" rpy="0 0 0"/>
+        </xacro:inertial_cylinder>
+    </link>
+    <!-- =========== END ARM =========== -->
+    <joint name="arm_joint_3" type="revolute">
+        <parent link="arm_2"/>
+        <child link="circuit_joint_3"/>
+        <origin xyz="0 0 0.55 " rpy="0 0 0"/> <!-- arm_2/2 1.1/2-->
+        <axis xyz="1 0 0"/>
+        <limit lower="-2.356" upper="2.356"
+           effort="10" velocity="1.0"/>
+    </joint>
+    <link name="circuit_joint_3">
+        <visual>
+            <origin xyz="0 0 0" rpy="0 1.5708 0"/>
+            <geometry>
+                <cylinder radius="0.2" length="0.3"/>
+            </geometry>
+            <material name="blue"/>
+        </visual>
+        <collision>
+            <origin xyz="0 0 0" rpy="0 1.5708 0"/>
+            <geometry>
+                <cylinder radius="0.2" length="0.3"/>
+            </geometry>
+        </collision>
+        <xacro:inertial_cylinder mass="0.1" radius="0.2" length="0.3">
+            <origin xyz="0 0 0" rpy="0 1.5708 0"/>
+        </xacro:inertial_cylinder>
+    </link>
+    <joint name="arm_joint_3_fixed" type="fixed">
+        <parent link="circuit_joint_3"/>
+        <child link="arm_3"/>
+        <origin xyz="0 0 0.35"/> <!-- circuit_joint_3/2 0.2/2 + arm_3/2 0.5/2-->
+    </joint>
+    <link name="arm_3">
+        <visual>
+            <origin xyz="0 0 0" rpy="0 0 0"/>
+            <geometry>
+                <cylinder radius="0.1" length="0.55"/>
+            </geometry>
+            <material name="blue"/>
+        </visual>
+        <collision>
+            <origin xyz="0 0 0" rpy="0 0 0"/>
+            <geometry>
+                <cylinder radius="0.1" length="0.5"/>
+            </geometry>
+        </collision>
+        <xacro:inertial_cylinder mass="0.1" radius="0.1" length="1.2">
+            <origin xyz="0 0 0" rpy="0 0 0"/>
         </xacro:inertial_cylinder>
     </link>
